Commit message: Started with ros

File: description/robot.urdf.xacro (robot description, xacro)
@@ -1,6 +1,4 @@
 <?xml version="1.0"?>
 <robot xmlns:xacro="http://www.ros.org/wiki/xacro"  name="robot">
-    <xacro:include filename="$(find ros_bot)/description/robot_core.xacro" />
-    <xacro:include filename="$(find ros_bot)/description/gazebo_control.xacro" />
-    <xacro:include filename="$(find ros_bot)/description/ros2_control.xacro" />
+    <xacro:include filename="$(find robotic_arm)/description/robot_core.xacro" />
 </robot>

File: description/robot_core.xacro (robot description, xacro)
@@ -1,33 +1,104 @@
 <?xml version="1.0"?>
-<robot xmlns:xacro="http://www.ros.org/wiki/xacro">
-    <xacro:include filename="$(find ros_bot)/description/inertial_macros.xacro"/>
-    <!-- BASE LINK -->
-    <link name="base_link"></link>
-    <!-- CHASSIS LINK -->
-    <joint name="chassis_joint" type="fixed">
-        <parent link="base_link"/>
-        <child link="chassis"/>
-        <origin xyz="0 0 0" rpy="0 0 0"/>
-    </joint>
-    <link name="chassis">
+<robot name="robotic_arm" xmlns:xacro="http://www.ros.org/wiki/xacro">
+    <!-- ================= BASE ================= -->
+    <link name="base_link">
         <visual>
             <origin xyz="0 0 0" rpy="0 0 0"/>
             <geometry>
-                <mesh filename="file://$(find ros_bot)/meshes/chassis.stl" scale="0.001 0.001 0.001"/>
+                <mesh filename="file://$(find robotic_arm)/meshes/base.stl" scale="0.001 0.001 0.001"/>
             </geometry>
-            <material name="">
+            <material name="white">
+                <color rgba="1 1 1 1"/>
+            </material>
+        </visual>
+        <collision>
+            <origin xyz="0 0 0" rpy="0 0 0"/>
+            <geometry>
+                <mesh filename="file://$(find robotic_arm)/meshes/base.stl" scale="0.001 0.001 0.001"/>
+            </geometry>
+        </collision>
+    </link>
+    <!-- ================= LINK 1 ================= -->
+    <joint name="joint1" type="revolute">
+        <parent link="base_link"/>
+        <child link="link1"/>
+        <!-- CHANGE THIS -->
+        <origin xyz="0 0 0.05" rpy="0 0 0"/>
+        <!-- ROTATION AXIS -->
+        <axis xyz="0 0 1"/>
+        <limit lower="-3.14"
+               upper="3.14"
+               effort="10"
+               velocity="1"/>
+    </joint>
+    <link name="link1">
+        <visual>
+            <origin xyz="0 0 0" rpy="0 0 0"/>
+            <geometry>
+                <mesh filename="file://$(find robotic_arm)/meshes/base_joint.stl"
+                      scale="0.001 0.001 0.001"/>
+            </geometry>
+            <material name="blue">
+                <color rgba="0 0 1 1"/>
             </material>
         </visual>
         <collision>
             <geometry>
-                <mesh filename="file://$(find ros_bot)/meshes/chassis.stl" scale="0.001 0.001 0.001"/>
+                <mesh filename="file://$(find robotic_arm)/meshes/base_joint.stl"
+                      scale="0.001 0.001 0.001"/>
             </geometry>
         </collision>
-        <xacro:inertial_box mass="1.0" x="0.24" y="0.18" z="0.04">
-            <origin xyz="0 0 0" rpy="0 0 0"/>
-        </xacro:inertial_box>
     </link>
-    <gazebo reference="chassis">
-        <material>Gazebo/White</material>
-    </gazebo>
+    <!-- ================= LINK 2 ================= -->
+    <joint name="joint2" type="revolute">
+        <parent link="link1"/>
+        <child link="link2"/>
+        <!-- CHANGE THIS -->
+        <origin xyz="0 0 0.05" rpy="0 0 0"/>
+        <axis xyz="0 1 0"/>
+        <limit lower="-1.57"
+               upper="1.57"
+               effort="10"
+               velocity="1"/>
+    </joint>
+    <link name="link2">
+        <visual>
+            <geometry>
+                <mesh filename="file://$(find robotic_arm)/meshes/arm1.stl"
+                      scale="0.001 0.001 0.001"/>
+            </geometry>
+        </visual>
+        <collision>
+            <geometry>
+                <mesh filename="file://$(find robotic_arm)/meshes/arm1.stl"
+                      scale="0.001 0.001 0.001"/>
+            </geometry>
+        </collision>
+    </link>
+    <!-- ================= LINK 3 ================= -->
+    <joint name="joint3" type="revolute">
+        <parent link="link2"/>
+        <child link="link3"/>
+        <!-- CHANGE THIS -->
+        <origin xyz="0 0 0.02" rpy="0 0 0"/>
+        <axis xyz="0 1 0"/>
+        <limit lower="-1.57"
+               upper="1.57"
+               effort="10"
+               velocity="1"/>
+    </joint>
+    <link name="link3">
+        <visual>
+            <geometry>
+                <mesh filename="file://$(find robotic_arm)/meshes/arm2.stl"
+                      scale="0.001 0.001 0.001"/>
+            </geometry>
+        </visual>
+        <collision>
+            <geometry>
+                <mesh filename="file://$(find robotic_arm)/meshes/arm2.stl"
+                      scale="0.001 0.001 0.001"/>
+            </geometry>
+        </collision>
+    </link>
 </robot>
